File: NixiePowerSupply.sch (KiCad schematic (older format))
At the start: 22 parts, among them J1 BARREL_JACK, J2 CONN_01X04, J3 CONN_01X05, Q1 2SA1015, Q2 2SK3234, U1 NJM2360, U2 Regul_7805

Commit message: first gerber out
Parts:
- Q2: value 2SK3234 -> 2SK3115
- U1: value NJM2360 -> MC34063A
Changed lines of the file:
@@
 P 4250 3900
 F 0 "U1" H 4050 4300 60  0000 C CNN
-F 1 "NJM2360" H 4250 3550 60  0000 C CNN
+F 1 "MC34063A" H 4250 3550 60  0000 C CNN
 F 2 "Housings_DIP:DIP-8_W7.62mm" H 4300 3900 60  0001 C CNN
 F 3 "" H 4300 3900 60  0001 C CNN
@@
 P 6000 3650
 F 0 "Q2" H 6200 3700 50  0000 L CNN
-F 1 "2SK3234" H 6200 3600 50  0000 L CNN
+F 1 "2SK3115" H 6200 3600 50  0000 L CNN
 F 2 "TO_SOT_Packages_THT:TO-220-3_Vertical" H 6200 3750 50  0001 C CNN
 F 3 "" H 6000 3650 50  0001 C CNN
